File: protoboard.brd (EAGLE design)
At the start: 99.1 x 48.3 mm, 118 parts, among them J3 AVX_6-PIN_009159006061916, J4 CORTEX_DEBUG_PTH, J5 10118194-0001LF, U1 STM32F103C8T6, U2 CJT1117-3.3-SOT223

Commit message: Added screenshots.
Parts:
- moved FRAME2 58.2 mm to (0.00, 0.00)
Routing:
- net PA1: track 24.8 -> 26.1 mm
- net PA3: track 47.1 -> 46.5 mm
- net PB8*: track 10.8 -> 11.3 mm
Other:
- board text added: "-------POWER------- VDD/AVDD: 2-3.6V. Must be 3.3V if C39- 097/C387- 415 are used for Q1/Q2. VUSB: 5V from USB (J5) VIN: 4.8-15V BAT: 1.8-3.6V. Short R2 if unused. ***WARNING***: Do NOT power MCU from VDD if EITHER VIN or USB (J5) are also being used. --------GPIO-------- Max current, ea pin: 25 mA Max current, total: 150 mA OUT (minus MCU power, ~7 -50 mA) and 150 mA IN (minus MCU po- wer) Bar o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"
- board text removed: "-------POWER------- VDD/AVDD: 2-3.6V. Must be 3.3V if C39- 097/C387- 415 are used for Q1/Q2. VUSB: 5V from USB1 VIN: 4.8-15V BAT: 1.8-3.6V. Short R2 if unused. **WARNING**: Do NOT power MCU from VDD if EITHER VIN or USB1 are also being used. --------GPIO-------- Max current, ea pin: 25 mA Max current, total: 150 mA OUT (minus MCU power, ~7 -50 mA) and 150 mA IN (minus MCU po- wer) Bar on pin labe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"
Changed lines of the file:
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@@
 <setting verticaltext="up"/>
 </settings>
-<grid distance="50" unitdist="mil" unit="mil" style="lines" multiple="1" display="yes" altdistance="5" altunitdist="mil" altunit="mil"/>
+<grid distance="25" unitdist="mil" unit="mil" style="lines" multiple="1" display="yes" altdistance="5" altunitdist="mil" altunit="mil"/>
 <layers>
 <layer number="1" name="Top" color="4" fill="1" visible="yes" active="yes"/>
@@
                        415 are used
                        for Q1/Q2.
-VUSB: 5V from USB1
+VUSB: 5V from USB (J5)
 VIN: 4.8-15V
 BAT: 1.8-3.6V. Short
    R2 if unused.
-**WARNING**: Do
+***WARNING***: Do
 NOT power MCU from VDD
-if EITHER VIN or USB1 are
-also being used.
+if EITHER VIN or USB (J5)
+are also being used.
 --------GPIO--------
 Max current, ea pin: 25 mA
@@
 J3: Debug Edge connector
 J4: J-Link connector
+J5: USB micro-B; Amphe-
+   nol 10118194-0001LF
 Q1: 8MHz / 3.2x2.5mm
 Q2: 32.768kHz / 3.2x2.5mm
@@
 C3, C4, C5, C7-C11: 100nF
 R3, R5: 10k | R8, R9: 150R
-D1, D2: Shottky / SOD-123
-LED1, LED2: 0603
 R1: 1k5                  C6: 1uF
 C1, C2:                    10uF
-S1: SPST-NO / 5.1mmx5.1mm
-           R2: 0R |     R4, R6:   0R
-         (R4/6 pull   BOOT0
-         /BOOT1     to GND if
-         J6/J7        not used)</text>
+D1, D2: Shottky / SOD-123
+            LED1, LED2: 0603
+          R2: 0R |     R4: 0R
+          (use R4 in lieu of J6/J7)
+          S1: SP     ST-NO /
+          5.1x        5.1mm</text>
 <text x="56.515" y="32.385" size="0.8128" layer="25" ratio="6" rot="R270">PWR</text>
 <text x="56.515" y="29.21" size="0.8128" layer="25" ratio="6" rot="R270">USER</text>
@@
 <attribute name="VALUE" x="53.34" y="27.305" size="1.27" layer="27"/>
 </element>
-<element name="FRAME2" library="SparkFun-Aesthetics" package="DUMMY" value="FRAME-LETTERNO_PACKAGE" x="-10.795" y="-57.15" smashed="yes">
-<attribute name="DESIGNER" value="Nathan Jones" x="-10.795" y="-57.15" size="1.778" layer="27" display="off"/>
-<attribute name="VERSION" value="v01" x="-10.795" y="-57.15" size="1.778" layer="27" display="off"/>
+<element name="FRAME2" library="SparkFun-Aesthetics" package="DUMMY" value="FRAME-LETTERNO_PACKAGE" x="0" y="0" smashed="yes">
+<attribute name="DESIGNER" value="Nathan Jones" x="0" y="0" size="1.778" layer="27" display="off"/>
+<attribute name="VERSION" value="v01" x="0" y="0" size="1.778" layer="27" display="off"/>
 </element>
 <element name="U1" library="STM32F103C8T6" package="LQFP48-7X7MM" value="STM32F103C8T6" x="31.75" y="24.13" smashed="yes" rot="R180">
@@
 </element>
 <element name="J3" library="Debug-Edge_AVX-connectors" package="AVX_6-PIN_009159006061916_0" value="AVX_6-PIN_009159006061916" x="0" y="17.145" smashed="yes" rot="R270">
-<attribute name="NAME" x="1.77" y="20.785" size="0.8128" layer="25" ratio="6" rot="R180"/>
+<attribute name="NAME" x="3.31" y="21.125" size="0.8128" layer="25" ratio="6"/>
 </element>
 <element name="L1" library="OPL_Ferrite_and_Magnetic_Bead" package="L0805" package3d_urn="urn:adsk.eagle:package:8004624/1" value="470R-2A" x="40.005" y="28.575" smashed="yes" rot="R90">
@@
 <contactref element="U1" pad="44"/>
 <contactref element="R3" pad="2"/>
-<wire x1="32.5" y1="19.88" x2="32.5" y2="18.53" width="0.127" layer="1"/>
-<wire x1="32.5" y1="18.53" x2="32.385" y2="18.415" width="0.127" layer="1"/>
-<via x="32.385" y="18.415" extent="1-16" drill="0.35"/>
-<wire x1="32.385" y1="18.415" x2="33.02" y2="19.05" width="0.127" layer="16"/>
 <wire x1="44.45" y1="19.05" x2="45.085" y2="18.415" width="0.127" layer="16"/>
 <wire x1="47.61" y1="18.415" x2="47.625" y2="18.4" width="0.127" layer="1"/>
-<wire x1="33.02" y1="19.05" x2="44.45" y2="19.05" width="0.127" layer="16"/>
 <via x="45.085" y="18.415" extent="1-16" drill="0.35"/>
+<wire x1="34.925" y1="19.05" x2="44.45" y2="19.05" width="0.127" layer="16"/>
 <wire x1="45.085" y1="18.415" x2="47.61" y2="18.415" width="0.127" layer="1"/>
+<wire x1="32.5" y1="19.88" x2="32.5" y2="20.435" width="0.127" layer="1"/>
+<wire x1="32.5" y1="20.435" x2="33.02" y2="20.955" width="0.127" layer="1"/>
+<via x="33.02" y="20.955" extent="1-16" drill="0.35"/>
+<wire x1="33.02" y1="20.955" x2="34.925" y2="19.05" width="0.127" layer="16"/>
 </signal>
 <signal name="OSC_OUT">
@@
 <signal name="PA9*">
 <contactref element="U1" pad="30"/>
-<wire x1="27.5" y1="24.38" x2="26.42" y2="24.38" width="0.127" layer="1"/>
-<via x="22.225" y="28.575" extent="1-16" drill="0.35"/>
-<wire x1="20.32" y1="30.48" x2="22.225" y2="28.575" width="0.127" layer="16"/>
-<wire x1="26.42" y1="24.38" x2="22.225" y2="28.575" width="0.127" layer="1"/>
 <contactref element="J1" pad="15"/>
-<wire x1="20.32" y1="33.02" x2="20.32" y2="30.48" width="0.127" layer="16"/>
+<wire x1="20.32" y1="30.48" x2="20.32" y2="33.02" width="0.127" layer="16"/>
 <contactref element="J51" pad="2"/>
 <contactref element="J51" pad="1"/>
 <wire x1="20.32" y1="33.02" x2="20.32" y2="35.56" width="0.889" layer="16"/>
 <wire x1="20.32" y1="35.56" x2="20.32" y2="38.1" width="0.889" layer="16"/>
+<wire x1="27.5" y1="24.38" x2="26.42" y2="24.38" width="0.127" layer="1"/>
+<via x="22.86" y="27.94" extent="1-16" drill="0.35"/>
+<wire x1="22.86" y1="27.94" x2="20.32" y2="30.48" width="0.127" layer="16"/>
+<wire x1="26.42" y1="24.38" x2="22.86" y2="27.94" width="0.127" layer="1"/>
 </signal>
 <signal name="PA10*">
@@
 <contactref element="U1" pad="45"/>
 <wire x1="33" y1="19.88" x2="33.02" y2="19.86" width="0.127" layer="1"/>
-<wire x1="33.02" y1="19.86" x2="33.02" y2="18.415" width="0.127" layer="1"/>
-<via x="33.02" y="18.415" extent="1-16" drill="0.35"/>
-<wire x1="35.56" y1="15.875" x2="33.02" y2="18.415" width="0.127" layer="16"/>
 <contactref element="J2" pad="9"/>
-<wire x1="35.56" y1="15.24" x2="35.56" y2="15.875" width="0.127" layer="16"/>
 <contactref element="J64" pad="2"/>
 <contactref element="J64" pad="1"/>
 <wire x1="35.56" y1="10.16" x2="35.56" y2="12.7" width="0.889" layer="16"/>
 <wire x1="35.56" y1="12.7" x2="35.56" y2="15.24" width="0.889" layer="16"/>
+<wire x1="33" y1="19.88" x2="33" y2="19.03" width="0.127" layer="1"/>
+<wire x1="33" y1="19.03" x2="32.385" y2="18.415" width="0.127" layer="1"/>
+<via x="32.385" y="18.415" extent="1-16" drill="0.35"/>
+<wire x1="32.385" y1="18.415" x2="35.56" y2="15.24" width="0.127" layer="16"/>
 </signal>
 <signal name="PB9*">
@@
 <contactref element="U1" pad="11"/>
 <wire x1="36" y1="26.38" x2="35.27" y2="26.38" width="0.127" layer="1"/>
-<wire x1="35.27" y1="26.38" x2="34.925" y2="26.035" width="0.127" layer="1"/>
-<via x="34.925" y="26.035" extent="1-16" drill="0.35"/>
-<wire x1="34.925" y1="26.035" x2="38.735" y2="22.225" width="0.127" layer="16"/>
 <wire x1="38.735" y1="22.225" x2="42.545" y2="22.225" width="0.127" layer="16"/>
 <wire x1="48.26" y1="16.51" x2="42.545" y2="22.225" width="0.127" layer="16"/>
@@
 <wire x1="48.26" y1="15.24" x2="48.26" y2="12.7" width="0.889" layer="16"/>
 <wire x1="48.26" y1="12.7" x2="48.26" y2="10.16" width="0.889" layer="16"/>
+<wire x1="35.27" y1="26.38" x2="34.925" y2="26.035" width="0.127" layer="1"/>
+<wire x1="34.925" y1="26.035" x2="34.29" y2="26.035" width="0.127" layer="1"/>
+<via x="34.29" y="26.035" extent="1-16" drill="0.35"/>
+<wire x1="34.29" y1="26.035" x2="34.925" y2="26.035" width="0.127" layer="16"/>
+<wire x1="34.925" y1="26.035" x2="38.735" y2="22.225" width="0.127" layer="16"/>
 </signal>
 <signal name="PA2">
@@
 <wire x1="56.515" y1="15.875" x2="56.515" y2="27.305" width="0.127" layer="1"/>
 <contactref element="J2" pad="1"/>
-<wire x1="34.5" y1="28.38" x2="34.5" y2="29.42" width="0.127" layer="1"/>
 <wire x1="44.069" y1="30.226" x2="45.085" y2="29.21" width="0.127" layer="1"/>
-<wire x1="34.5" y1="29.42" x2="35.306" y2="30.226" width="0.127" layer="1"/>
-<wire x1="35.306" y1="30.226" x2="44.069" y2="30.226" width="0.127" layer="1"/>
+<wire x1="36.346" y1="30.226" x2="44.069" y2="30.226" width="0.127" layer="1"/>
 <wire x1="55.88" y1="15.24" x2="56.515" y2="15.875" width="0.127" layer="1"/>
 <contactref element="J80" pad="2"/>
@@
 <wire x1="55.88" y1="10.16" x2="55.88" y2="12.7" width="0.889" layer="16"/>
 <wire x1="55.88" y1="12.7" x2="55.88" y2="15.24" width="0.889" layer="16"/>
+<wire x1="34.5" y1="28.38" x2="36.346" y2="30.226" width="0.127" layer="1"/>
 </signal>
 <signal name="PA4">
 <contactref element="U1" pad="14"/>
-<wire x1="34" y1="28.38" x2="34" y2="29.555" width="0.127" layer="1"/>
-<wire x1="34" y1="29.555" x2="34.29" y2="29.845" width="0.127" layer="1"/>
-<via x="34.29" y="29.845" extent="1-16" drill="0.35"/>
-<wire x1="34.925" y1="30.48" x2="34.29" y2="29.845" width="0.127" layer="16"/>
 <contactref element="J1" pad="1"/>
 <wire x1="55.88" y1="33.02" x2="53.34" y2="30.48" width="0.127" layer="16"/>
-<wire x1="53.34" y1="30.48" x2="34.925" y2="30.48" width="0.127" layer="16"/>
+<wire x1="53.34" y1="30.48" x2="35.56" y2="30.48" width="0.127" layer="16"/>
 <contactref element="J79" pad="2"/>
 <contactref element="J79" pad="1"/>
 <wire x1="55.88" y1="33.02" x2="55.88" y2="35.56" width="0.889" layer="16"/>
 <wire x1="55.88" y1="35.56" x2="55.88" y2="38.1" width="0.889" layer="16"/>
+<wire x1="34" y1="28.38" x2="34" y2="28.92" width="0.127" layer="1"/>
+<wire x1="34" y1="28.92" x2="34.925" y2="29.845" width="0.127" layer="1"/>
+<via x="34.925" y="29.845" extent="1-16" drill="0.35"/>
+<wire x1="34.925" y1="29.845" x2="35.56" y2="30.48" width="0.127" layer="16"/>
 </signal>
 <signal name="PA5">
