File: protoboard.sch (EAGLE design)
At the start: 118 parts, among them J3 AVX_6-PIN_009159006061916, J4 CORTEX_DEBUG_PTH, J5 10118194-0001LF, U1 STM32F103C8T6, U2 CJT1117-3.3-SOT223

Commit message: Updated design block. Switched USB from micro-B to mini-B. Updated Debug Edge library.
Parts:
- removed C1, C2: 10uF, adafruit:C-USC0402
- removed C10, C11, C3, C4, C5, C7, C8, C9: 100nF, adafruit:C-USC0402
- removed C6: 1uF, adafruit:C-USC0402
- removed D1, D2: (no value), adafruit:DIODESOD-123
- removed FRAME2: FRAME-LETTERNO_PACKAGE, SparkFun-Aesthetics:FRAME-LETTERNO_PACKAGE
- removed J1, J2: (no value), SparkFun-Connectors:CONN_20NOSILK
- removed J3: AVX_6-PIN_009159006061916, Debug-Edge_AVX-connectors:AVX_6-PIN_009159006061916
- removed J4: CORTEX_DEBUG_PTH, SparkFun-Connectors:CORTEX_DEBUG_PTH
- removed J5: 10118194-0001LF, USB-micro-B_Amphenol_10118194-0001LF:10118194-0001LF
- removed J6, J7: (no value), SparkFun-Connectors:CONN_031X03_NO_SILK
- removed J8: (no value), SparkFun-Connectors:CONN_021X02_NO_SILK
- removed L1: 470R-2A, OPL_Ferrite_and_Magnetic_Bead:SMD-FERRITE-BEAD-470R-2A(0805)'0805'
- removed LED1, LED2: (no value), adafruit:LEDCHIPLED_0603
- removed Q1, Q2: (no value), crystal-geyer_V1_0:KXO-VCXO-CMOS_4
- removed R1: 1k5, adafruit:R-US_R0402
- removed R2, R4, R6: 0R, adafruit:R-US_R0402
- removed R3, R5: 10k, adafruit:R-US_R0402
- removed R7, R8: 150R, adafruit:R-US_R0402
- removed S1: MOMENTARY-SWITCH-SPST-SMD-5.2-REDUNDANT, SparkFun-Switches:MOMENTARY-SWITCH-SPST-SMD-5.2-REDUNDANT
- removed U1: STM32F103C8T6, STM32F103C8T6:STM32F103C8T6
- removed U2: CJT1117-3.3-SOT223, OPL_IC:PMIC-CJT1117-3.3(SOT223)
- added C12, C13: 10uF, SparkFun-Capacitors:0.1UF-0402T-16V-10%
- added C14, C15, C16, C18, C19, C20, C21, C22: 100nF, SparkFun-Capacitors:0.1UF-0402T-16V-10%
- added C17: 1uF, SparkFun-Capacitors:0.1UF-0402T-16V-10%
- added D3, D4: (no value), adafruit:DIODESOD-123
- added FRAME1: FRAME-LETTERNO_PACKAGE, SparkFun-Aesthetics:FRAME-LETTERNO_PACKAGE
- added J82: CORTEX_DEBUG_PTH, SparkFun-Connectors:CORTEX_DEBUG_PTH
- added J83, J84: (no value), SparkFun-Connectors:CONN_031X03_NO_SILK
- added J85: (no value), SparkFun-Connectors:CONN_021X02_NO_SILK
- added J86: (no value), SparkFun-Connectors:CONN_20NOSILK
- added J87, J88: (no value), SparkFun-Connectors:CONN_111X11_NO_SILK
- added J97: 2172034-1, 2172034-1:2172034-1
- added J98: AVX_6-PIN_009159006061916_33MIL-GAP, Debug-Edge_AVX-connectors:AVX_6-PIN_009159006061916_33MIL-GAP
- added L2: 470R-2A, OPL_Ferrite_and_Magnetic_Bead:SMD-FERRITE-BEAD-470R-2A(0805)'0805'
- added LED3, LED4: (no value), adafruit:LEDCHIPLED_0603
- added Q3, Q4: (no value), crystal-geyer_V1_0:KXO-VCXO-CMOS_4
- added R10, R12, R14: 0R, SparkFun-Resistors:RESISTOR0402
- added R11, R13: 10k, SparkFun-Resistors:RESISTOR0402
- added R15, R16: 150R, SparkFun-Resistors:RESISTOR0402
- added R9: 1k5, SparkFun-Resistors:RESISTOR0402
- added S2: MOMENTARY-SWITCH-SPST-SMD-5.2-REDUNDANT, SparkFun-Switches:MOMENTARY-SWITCH-SPST-SMD-5.2-REDUNDANT
- added U3: STM32F103C8T6, STM32F103C8T6:STM32F103C8T6
- added U4: CJT1117-3.3-SOT223, OPL_IC:PMIC-CJT1117-3.3(SOT223)
Connections:
- removed net N$21: J13.1, J13.2
- removed net N$24: J15.1, J15.2
- removed net N$81: J6.2, R3.1, R4.2
- removed net N$82: J7.2, R5.1, R6.2
- removed net N$83: LED2.A, R8.2
- removed net N$84: LED1.A, R7.1
- removed net VIN: C1.1, D1.C, D2.C, U2.IN
- new net N$58: J83.2, R11.1, R12.2
- new net N$59: J84.2, R13.1, R14.2
- new net N$60: LED4.A, R16.1
- new net N$61: LED3.A, R15.1
- new net VIN2: C12.1, D3.C, D4.C, U4.IN
- net AVDD: now also C17.1, C18.1, J86.2, L2.1, U3B.VDDA; no longer C6.1, C7.1, J2.2, L1.1, U1B.VDDA
- net BOOT0: now also R11.2, U3A.BOOT0; no longer R3.2, U1A.BOOT0
- net BOOT1*: now also J87.7, R13.2, U3A.PB2; no longer J1.7, R5.2, U1A.PB2
- net GND: now also C12.2, C13.2, C14.2, C15.2, C16.2, C17.2, C18.2, C19.2, C20.2, C21.2, C22.2, J13.1, J13.2, J15.1, J15.2, J82.GND@3, J82.GND@5, J83.1, J84.1, J86.18, J88.10, J88.11, J97.4, J97.5, J97.MH1, J97.MH2, J98.6, LED3.C, LED4.C, Q3.GND, Q4.GND, R12.1, R14.1, S2.1, U3B.VSSA, U3B.VSS_1, U3B.VSS_2, U3B.VSS_3, U4.GND; no longer C1.2, C10.2, C11.2, C2.2, C3.2, C4.2, C5.2, C6.2, C7.2, C8.2, C9.2, J2.18, J3.6, J4.GND@3, J4.GND@5, J5.4, J5.5, J6.1, J7.1, LED1.C, LED2.C, Q1.GND, Q2.GND, R4.1, R6.1, S1.1, U1B.VSSA, U1B.VSS_1, U1B.VSS_2, U1B.VSS_3, U2.GND
- net JTDI*: now also J82.NC/TDI, J86.14, U3A.PA15; no longer J2.14, J4.NC/TDI, U1A.PA15
- net JTRST*: now also J82.GNDDTCT, J86.13, U3A.PB4; no longer J2.13, J4.GNDDTCT, U1A.PB4
- net NRST: now also C20.1, J82.!RESET, J86.15, J98.5, S2.2, U3A.NRST; no longer C9.1, J2.15, J3.5, J4.!RESET, S1.2, U1A.NRST
- net OSC32_IN: now also Q4.OUT, U3A.PC14-OSC32_IN; no longer Q2.OUT, U1A.PC14-OSC32_IN
- net OSC32_OUT: now also U3A.PC15-OSC32_OUT; no longer U1A.PC15-OSC32_OUT
- net OSC_IN: now also Q3.OUT, U3A.OSC_IN; no longer Q1.OUT, U1A.OSC_IN
- net OSC_OUT: now also U3A.OSC_OUT; no longer U1A.OSC_OUT
- net PA0: now also J86.5, U3A.PA0-WKUP; no longer J2.5, U1A.PA0-WKUP
- net PA1: now also J86.4, U3A.PA1; no longer J2.4, U1A.PA1
- net PA10*: now also J88.5, U3A.PA10; no longer J1.16, U1A.PA10
- net PA2: now also J86.3, U3A.PA2; no longer J2.3, U1A.PA2
- net PA3: now also J85.1, J85.2, J86.1, R16.2, U3A.PA3; no longer J2.1, J8.1, J8.2, R8.1, U1A.PA3
- net PA4: now also J87.1, U3A.PA4; no longer J1.1, U1A.PA4
- net PA5: now also J87.2, U3A.PA5; no longer J1.2, U1A.PA5
- net PA6: now also J87.3, U3A.PA6; no longer J1.3, U1A.PA6
- net PA7: now also J87.4, U3A.PA7; no longer J1.4, U1A.PA7
- net PA8*: now also J88.3, U3A.PA8; no longer J1.14, U1A.PA8
- net PA9*: now also J88.4, U3A.PA9; no longer J1.15, U1A.PA9
- net PB0: now also J87.5, U3A.PB0; no longer J1.5, U1A.PB0
- net PB1: now also J87.6, U3A.PB1; no longer J1.6, U1A.PB1
- net PB10*: now also J87.8, U3A.PB10; no longer J1.8, U1A.PB10
- net PB11*: now also J87.9, U3A.PB11; no longer J1.9, U1A.PB11
- net PB12*: now also J87.10, U3A.PB12; no longer J1.10, U1A.PB12
- net PB13*: now also J87.11, U3A.PB13; no longer J1.11, U1A.PB13
- net PB14*: now also J88.1, U3A.PB14; no longer J1.12, U1A.PB14
- net PB15*: now also J88.2, U3A.PB15; no longer J1.13, U1A.PB15
- net PB5: now also J86.12, U3A.PB5; no longer J2.12, U1A.PB5
- net PB6*: now also J86.11, U3A.PB6; no longer J2.11, U1A.PB6
- net PB7*: now also J86.10, U3A.PB7; no longer J2.10, U1A.PB7
- net PB8*: now also J86.9, U3A.PB8; no longer J2.9, U1A.PB8
- net PB9*: now also J86.8, U3A.PB9; no longer J2.8, U1A.PB9
- net PC13: now also J86.6, U3A.PC13; no longer J2.6, U1A.PC13
- net SWCLK*: now also J82.SWDCLK/TCK, J86.19, J98.2, U3A.PA14; no longer J2.19, J3.2, J4.SWDCLK/TCK, U1A.PA14
- net SWDIO*: now also J82.SWDIO/TMS, J86.17, J98.1, U3A.PA13; no longer J2.17, J3.1, J4.SWDIO/TMS, U1A.PA13
- net SWO*: now also J82.SWO/TDO, J86.16, J98.3, U3A.PB3; no longer J2.16, J3.3, J4.SWO/TDO, U1A.PB3
- net USB_DM*: now also J19.1, J19.2, J88.8, J97.2, U3A.PA11; no longer J1.18, J45.1, J45.2, J5.2, U1A.PA11
- net USB_DP*: now also J17.1, J17.2, J88.9, J97.3, R9.1, U3A.PA12; no longer J1.19, J19.1, J19.2, J5.3, R1.1, U1A.PA12
- net VBAT_1.8-3.6V: now also C19.1, J86.7, R10.1, U3B.VBAT; no longer C8.1, J2.7, R2.1, U1B.VBAT
- net VDD: now also C13.1, C14.1, C15.1, C16.1, C21.1, C22.1, J82.VCC, J83.3, J84.3, J86.20, J98.4, L2.2, Q3.VDD, Q4.VDD, R10.2, R15.2, R9.2, U3B.VDD_1, U3B.VDD_2, U3B.VDD_3, U4.OUT; no longer C10.1, C11.1, C2.1, C3.1, C4.1, C5.1, J2.20, J3.4, J4.VCC, J6.3, J7.3, L1.2, Q1.VDD, Q2.VDD, R1.2, R2.2, R7.2, U1B.VDD_1, U1B.VDD_2, U1B.VDD_3, U2.OUT
- net VIN_4.8-15V: now also D4.A, J88.6; no longer D2.A, J1.17
- net VUSB: now also D3.A, J45.1, J45.2, J88.7, J97.1; no longer D1.A, J1.20, J17.1, J17.2, J5.1
